File: pinout.kicad_sch (KiCad schematic)
At the start: 57 parts

Commit message: relabel components by sheet and block
Parts:
- renumbered TP68 to TP25, TP69 to TP26, TP70 to TP27, TP71 to TP28, TP25 to TP29, TP37 to TP30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
