File: f405-fc-mcu_sch.kicad_sch (KiCad schematic)
At the start: 27 parts, among them U1 STM32F405RGTx, Y1 8MHz

Commit message: replace flash memory with SD flash memory; move SPI2 terminations closer to source
Parts:
- C1: Manufactorer Samsung -> Murata; Part Number CL21A106KBYQNNE -> GRM21BR61H106KE43K
- C10, C2, C3, C4, C5, C6, C7: Part Number CC0402KRX7R7BB104 -> CC0402KRX5R8BB104; Voltage 16 -> 25
- C11, C12: Part Number GRM188C71C225KE11D -> GRM188R61E225KA12D; Voltage 16 -> 25
- C13, C14: Voltage 16 -> 50
- C8, C9: Voltage 16 -> 25
- FB1: Voltage (none) -> 2.5
- SW1: value ~ -> EVP-AA602W; Manufactorer (none) -> Panasonic; Part Number (none) -> EVP-AA602W
Changed lines of the file:
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@@
 			)
 		)
-		(property "Part Number" "CC0402KRX7R7BB104"
+		(property "Part Number" "CC0402KRX5R8BB104"
 			(at 171.45 43.18 0)
 			(effects
@@
 			)
 		)
-		(property "Voltage" "16"
+		(property "Voltage" "25"
 			(at 171.45 43.18 0)
 			(effects
@@
 			)
 		)
-		(property "Voltage" "16"
+		(property "Voltage" "25"
 			(at 104.14 43.18 0)
 			(effects
@@
 			)
 		)
-		(property "Part Number" "CC0402KRX7R7BB104"
+		(property "Part Number" "CC0402KRX5R8BB104"
 			(at 104.14 43.18 0)
 			(effects
@@
 			)
 		)
-		(property "Voltage" "16"
+		(property "Voltage" "25"
 			(at 119.38 43.18 0)
 			(effects
@@
 			)
 		)
-		(property "Part Number" "CC0402KRX7R7BB104"
+		(property "Part Number" "CC0402KRX5R8BB104"
 			(at 119.38 43.18 0)
 			(effects
@@
 			)
 		)
-		(property "Voltage" "16"
+		(property "Voltage" "25"
 			(at 191.77 43.18 0)
 			(effects
@@
 			)
 		)
-		(property "Voltage" "16"
+		(property "Voltage" "25"
 			(at 48.26 60.96 0)
 			(effects
@@
 			)
 		)
-		(property "Part Number" "CC0402KRX7R7BB104"
+		(property "Part Number" "CC0402KRX5R8BB104"
 			(at 48.26 60.96 0)
 			(effects
@@
 			)
 		)
-		(property "Voltage" "16"
+		(property "Voltage" "25"
 			(at 179.07 43.18 0)
 			(effects
@@
 			)
 		)
-		(property "Voltage" "16"
+		(property "Voltage" "50"
 			(at 62.23 171.45 0)
 			(effects
@@
 			)
 		)
-		(property "Voltage" "16"
+		(property "Voltage" "25"
 			(at 111.76 43.18 0)
 			(effects
@@
 			)
 		)
-		(property "Part Number" "CC0402KRX7R7BB104"
+		(property "Part Number" "CC0402KRX5R8BB104"
 			(at 111.76 43.18 0)
 			(effects
@@
 			)
 		)
-		(property "Voltage" "16"
+		(property "Voltage" "25"
 			(at 116.84 129.54 0)
 			(effects
@@
 			)
 		)
-		(property "Part Number" "GRM188C71C225KE11D"
+		(property "Part Number" "GRM188R61E225KA12D"
 			(at 116.84 129.54 0)
 			(effects
@@
 			)
 		)
-		(property "Manufactorer" "Samsung"
+		(property "Manufactorer" "Murata"
 			(at 88.9 43.18 0)
 			(effects
@@
 			)
 		)
-		(property "Part Number" "CL21A106KBYQNNE"
+		(property "Part Number" "GRM21BR61H106KE43K"
 			(at 88.9 43.18 0)
 			(effects
@@
 			)
 		)
-		(property "Voltage" "16"
+		(property "Voltage" "25"
 			(at 128.27 129.54 0)
 			(effects
@@
 			)
 		)
-		(property "Part Number" "GRM188C71C225KE11D"
+		(property "Part Number" "GRM188R61E225KA12D"
 			(at 128.27 129.54 0)
 			(effects
@@
 			)
 		)
-		(property "Voltage" "16"
+		(property "Voltage" "25"
 			(at 127 43.18 0)
 			(effects
@@
 			)
 		)
-		(property "Part Number" "CC0402KRX7R7BB104"
+		(property "Part Number" "CC0402KRX5R8BB104"
 			(at 127 43.18 0)
 			(effects
@@
 			)
 		)
-		(property "Datasheet" "~"
+		(property "Datasheet" "https://ecsxtal.com/store/pdf/ecx-32.pdf"
 			(at 53.34 161.29 0)
 			(effects
@@
 			)
 		)
-		(property "Value" "~"
+		(property "Value" "EVP-AA602W"
 			(at 88.9 57.15 0)
 			(effects
@@
 			)
 		)
-		(property "Datasheet" "EVP-AA602W"
+		(property "Datasheet" "https://www3.panasonic.biz/ac/cdn/e/control/switch/light-touch/catalog/sw_lt_eng_3529s.pdf"
 			(at 93.98 62.23 0)
 			(effects
@@
 			)
 		)
+		(property "Manufactorer" "Panasonic"
+			(at 93.98 62.23 0)
+			(effects
+				(font
+					(size 1.27 1.27)
+				)
+				(hide yes)
+			)
+		)
+		(property "Part Number" "EVP-AA602W"
+			(at 93.98 62.23 0)
+			(effects
+				(font
+					(size 1.27 1.27)
+				)
+				(hide yes)
+			)
+		)
 		(pin "4"
 		)
@@
 			)
 		)
-		(property "Voltage" "16"
+		(property "Voltage" "50"
 			(at 43.18 171.45 0)
 			(effects
@@
 			)
 		)
-		(property "Datasheet" "~"
+		(property "Datasheet" "https://www.laird.com/sites/default/files/mi0603m121r-10-datasheet.pdf"
 			(at 185.42 38.1 0)
 			(effects
@@
 			)
 		)
+		(property "Voltage" "2.5"
+			(at 185.42 38.1 0)
+			(effects
+				(font
+					(size 1.27 1.27)
+				)
+				(hide yes)
+			)
+		)
 		(pin "1"
 		)
@@
 			)
 		)
-		(property "Voltage" "16"
+		(property "Voltage" "25"
 			(at 96.52 43.18 0)
 			(effects
@@
 			)
 		)
-		(property "Part Number" "CC0402KRX7R7BB104"
+		(property "Part Number" "CC0402KRX5R8BB104"
 			(at 96.52 43.18 0)
 			(effects

Commit message: remove blind vias and use 0201 resistors
Parts:
- C10, C2, C3, C4, C5, C6, C7: footprint Capacitor_SMD:C_0402_1005Metric -> Project:C_0201_0603Metric; Manufactorer YAGEO -> Murata; Part Number CC0402KRX5R8BB104 -> GRM033R61E104KE14J
- C11, C12: footprint Capacitor_SMD:C_0603_1608Metric -> Capacitor_SMD:C_0402_1005Metric; Manufactorer Murata -> YAGEO; Part Number GRM188R61E225KA12D -> CC0402KPX5R8BB225
- C13, C14: Manufactorer YAGEO -> Murata; Part Number CC0402GRNPO9BN160 -> GCM1555C1H160FA16D
- C8, C9: value 1u -> 2u2; footprint Capacitor_SMD:C_0603_1608Metric -> Capacitor_SMD:C_0402_1005Metric; Part Number CC0603KRX5R8BB105 -> CC0402KPX5R8BB225
- R1: value 22k -> 22k1; footprint Resistor_SMD:R_0402_1005Metric -> Project:R_0201_0603Metric; Part Number RC0402FR-0722KL -> RC0201FR-0722K1L
- R2, R3, R8, R9: footprint Resistor_SMD:R_0402_1005Metric -> Project:R_0201_0603Metric; Part Number RC0402FR-0722RP -> RC0201FR-0722RL
- R4, R5, R6, R7: footprint Resistor_SMD:R_0402_1005Metric -> Project:R_0201_0603Metric; Part Number RC0402FR-075K1L -> RC0201FR-075K1L
Changed lines of the file:
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@@
 			)
 		)
-		(property "Footprint" "Capacitor_SMD:C_0402_1005Metric"
+		(property "Footprint" "Project:C_0201_0603Metric"
 			(at 172.4152 46.99 0)
 			(effects
@@
 			)
 		)
-		(property "Manufactorer" "YAGEO"
+		(property "Manufactorer" "Murata"
 			(at 171.45 43.18 0)
 			(effects
@@
 			)
 		)
-		(property "Part Number" "CC0402KRX5R8BB104"
+		(property "Part Number" "GRM033R61E104KE14J"
 			(at 171.45 43.18 0)
 			(effects
@@
 			)
 		)
-		(property "Footprint" "Capacitor_SMD:C_0402_1005Metric"
+		(property "Footprint" "Project:C_0201_0603Metric"
 			(at 105.1052 46.99 0)
 			(effects
@@
 			)
 		)
-		(property "Manufactorer" "YAGEO"
+		(property "Manufactorer" "Murata"
 			(at 104.14 43.18 0)
 			(effects
@@
 			)
 		)
-		(property "Part Number" "CC0402KRX5R8BB104"
+		(property "Part Number" "GRM033R61E104KE14J"
 			(at 104.14 43.18 0)
 			(effects
@@
 			)
 		)
-		(property "Footprint" "Resistor_SMD:R_0402_1005Metric"
+		(property "Footprint" "Project:R_0201_0603Metric"
 			(at 195.58 140.208 90)
 			(effects
@@
 			)
 		)
-		(property "Part Number" "RC0402FR-0722RP"
+		(property "Part Number" "RC0201FR-0722RL"
 			(at 195.58 138.43 0)
 			(effects
@@
 			)
 		)
-		(property "Footprint" "Resistor_SMD:R_0402_1005Metric"
+		(property "Footprint" "Project:R_0201_0603Metric"
 			(at 216.662 111.76 90)
 			(effects
@@
 			)
 		)
-		(property "Part Number" "RC0402FR-075K1L"
+		(property "Part Number" "RC0201FR-075K1L"
 			(at 218.44 111.76 0)
 			(effects
@@
 			)
 		)
-		(property "Footprint" "Resistor_SMD:R_0402_1005Metric"
+		(property "Footprint" "Project:R_0201_0603Metric"
 			(at 199.39 71.628 90)
 			(effects
@@
 			)
 		)
-		(property "Part Number" "RC0402FR-0722RP"
+		(property "Part Number" "RC0201FR-0722RL"
 			(at 199.39 69.85 0)
 			(effects
@@
 			)
 		)
-		(property "Value" "22k"
+		(property "Value" "22k1"
 			(at 106.68 67.31 0)
 			(effects
@@
 			)
 		)
-		(property "Footprint" "Resistor_SMD:R_0402_1005Metric"
+		(property "Footprint" "Project:R_0201_0603Metric"
 			(at 102.362 66.04 90)
 			(effects
@@
 			)
 		)
-		(property "Part Number" "RC0402FR-0722KL"
+		(property "Part Number" "RC0201FR-0722K1L"
 			(at 104.14 66.04 0)
 			(effects
@@
 			)
 		)
-		(property "Footprint" "Capacitor_SMD:C_0402_1005Metric"
+		(property "Footprint" "Project:C_0201_0603Metric"
 			(at 120.3452 46.99 0)
 			(effects
@@
 			)
 		)
-		(property "Manufactorer" "YAGEO"
+		(property "Manufactorer" "Murata"
 			(at 119.38 43.18 0)
 			(effects
@@
 			)
 		)
-		(property "Part Number" "CC0402KRX5R8BB104"
+		(property "Part Number" "GRM033R61E104KE14J"
 			(at 119.38 43.18 0)
 			(effects
@@
 			)
 		)
-		(property "Footprint" "Resistor_SMD:R_0402_1005Metric"
+		(property "Footprint" "Project:R_0201_0603Metric"
 			(at 199.39 76.708 90)
 			(effects
@@
 			)
 		)
-		(property "Part Number" "RC0402FR-0722RP"
+		(property "Part Number" "RC0201FR-0722RL"
 			(at 199.39 74.93 0)
 			(effects
@@
 			)
 		)
-		(property "Value" "1u"
+		(property "Value" "2u2"
 			(at 195.58 44.45 0)
 			(effects
@@
 			)
 		)
-		(property "Footprint" "Capacitor_SMD:C_0603_1608Metric"
+		(property "Footprint" "Capacitor_SMD:C_0402_1005Metric"
 			(at 192.7352 46.99 0)
 			(effects
@@
 			)
 		)
-		(property "Part Number" "CC0603KRX5R8BB105"
+		(property "Part Number" "CC0402KPX5R8BB225"
 			(at 191.77 43.18 0)
 			(effects
@@
 			)
 		)
-		(property "Footprint" "Capacitor_SMD:C_0402_1005Metric"
+		(property "Footprint" "Project:C_0201_0603Metric"
 			(at 49.2252 64.77 0)
 			(effects
@@
 			)
 		)
-		(property "Manufactorer" "YAGEO"
+		(property "Manufactorer" "Murata"
 			(at 48.26 60.96 0)
 			(effects
@@
 			)
 		)
-		(property "Part Number" "CC0402KRX5R8BB104"
+		(property "Part Number" "GRM033R61E104KE14J"
 			(at 48.26 60.96 0)
 			(effects
@@
 			)
 		)
-		(property "Value" "1u"
+		(property "Value" "2u2"
 			(at 177.8 35.56 0)
 			(effects
@@
 			)
 		)
-		(property "Footprint" "Capacitor_SMD:C_0603_1608Metric"
+		(property "Footprint" "Capacitor_SMD:C_0402_1005Metric"
 			(at 180.0352 46.99 0)
 			(effects
@@
 			)
 		)
-		(property "Part Number" "CC0603KRX5R8BB105"
+		(property "Part Number" "CC0402KPX5R8BB225"
 			(at 179.07 43.18 0)
 			(effects
@@
 			)
 		)
-		(property "Footprint" "Resistor_SMD:R_0402_1005Metric"
+		(property "Footprint" "Project:R_0201_0603Metric"
 			(at 195.58 135.128 90)
 			(effects
@@
 			)
 		)
-		(property "Part Number" "RC0402FR-0722RP"
+		(property "Part Number" "RC0201FR-0722RL"
 			(at 195.58 133.35 0)
 			(effects
@@
 			)
 		)
-		(property "Manufactorer" "YAGEO"
+		(property "Manufactorer" "Murata"
 			(at 62.23 171.45 0)
 			(effects
@@
 			)
 		)
-		(property "Part Number" "CC0402GRNPO9BN160"
+		(property "Part Number" "GCM1555C1H160FA16D"
 			(at 62.23 171.45 0)
 			(effects
@@
 			)
 		)
-		(property "Footprint" "Capacitor_SMD:C_0402_1005Metric"
+		(property "Footprint" "Project:C_0201_0603Metric"
 			(at 112.7252 46.99 0)
 			(effects
@@
 			)
 		)
-		(property "Manufactorer" "YAGEO"
+		(property "Manufactorer" "Murata"
 			(at 111.76 43.18 0)
 			(effects
@@
 			)
 		)
-		(property "Part Number" "CC0402KRX5R8BB104"
+		(property "Part Number" "GRM033R61E104KE14J"
 			(at 111.76 43.18 0)
 			(effects
@@
 			)
 		)
-		(property "Footprint" "Capacitor_SMD:C_0603_1608Metric"
+		(property "Footprint" "Capacitor_SMD:C_0402_1005Metric"
 			(at 117.8052 133.35 0)
 			(effects
@@
 			)
 		)
-		(property "Manufactorer" "Murata"
+		(property "Manufactorer" "YAGEO"
 			(at 116.84 129.54 0)
 			(effects
@@
 			)
 		)
-		(property "Part Number" "GRM188R61E225KA12D"
+		(property "Part Number" "CC0402KPX5R8BB225"
 			(at 116.84 129.54 0)
 			(effects
@@
 			)
 		)
-		(property "Footprint" "Capacitor_SMD:C_0603_1608Metric"
+		(property "Footprint" "Capacitor_SMD:C_0402_1005Metric"
 			(at 129.2352 133.35 0)
 			(effects
@@
 			)
 		)
-		(property "Manufactorer" "Murata"
+		(property "Manufactorer" "YAGEO"
 			(at 128.27 129.54 0)
 			(effects
@@
 			)
 		)
-		(property "Part Number" "GRM188R61E225KA12D"
+		(property "Part Number" "CC0402KPX5R8BB225"
 			(at 128.27 129.54 0)
 			(effects
@@
 			)
 		)
-		(property "Footprint" "Resistor_SMD:R_0402_1005Metric"
+		(property "Footprint" "Project:R_0201_0603Metric"
 			(at 235.712 121.92 90)
 			(effects
@@
 			)
 		)
-		(property "Part Number" "RC0402FR-075K1L"
+		(property "Part Number" "RC0201FR-075K1L"
 			(at 237.49 121.92 0)
 			(effects
@@
 			)
 		)
-		(property "Footprint" "Capacitor_SMD:C_0402_1005Metric"
+		(property "Footprint" "Project:C_0201_0603Metric"
 			(at 127.9652 46.99 0)
 			(effects
@@
 			)
 		)
-		(property "Manufactorer" "YAGEO"
+		(property "Manufactorer" "Murata"
 			(at 127 43.18 0)
 			(effects
@@
 			)
 		)
-		(property "Part Number" "CC0402KRX5R8BB104"
+		(property "Part Number" "GRM033R61E104KE14J"
 			(at 127 43.18 0)
 			(effects
@@
 			)
 		)
-		(property "Footprint" "Resistor_SMD:R_0402_1005Metric"
+		(property "Footprint" "Project:R_0201_0603Metric"
 			(at 196.342 111.76 90)
 			(effects
@@
 			)
 		)
-		(property "Part Number" "RC0402FR-075K1L"
+		(property "Part Number" "RC0201FR-075K1L"
 			(at 198.12 111.76 0)
 			(effects
@@
 			)
 		)
-		(property "Manufactorer" "YAGEO"
+		(property "Manufactorer" "Murata"
 			(at 43.18 171.45 0)
 			(effects
@@
 			)
 		)
-		(property "Part Number" "CC0402GRNPO9BN160"
+		(property "Part Number" "GCM1555C1H160FA16D"
 			(at 43.18 171.45 0)
 			(effects
@@
 			)
 		)
-		(property "Footprint" "Resistor_SMD:R_0402_1005Metric"
+		(property "Footprint" "Project:R_0201_0603Metric"
 			(at 257.302 121.92 90)
 			(effects
@@
 			)
 		)
-		(property "Part Number" "RC0402FR-075K1L"
+		(property "Part Number" "RC0201FR-075K1L"
 			(at 259.08 121.92 0)
 			(effects
@@
 			)
 		)
-		(property "Footprint" "Capacitor_SMD:C_0402_1005Metric"
+		(property "Footprint" "Project:C_0201_0603Metric"
 			(at 97.4852 46.99 0)
 			(effects
@@
 			)
 		)
-		(property "Manufactorer" "YAGEO"
+		(property "Manufactorer" "Murata"
 			(at 96.52 43.18 0)
 			(effects
@@
 			)
 		)
-		(property "Part Number" "CC0402KRX5R8BB104"
+		(property "Part Number" "GRM033R61E104KE14J"
 			(at 96.52 43.18 0)
 			(effects

Commit message: double check BOM
Parts:
- C11, C12, C8, C9: Manufactorer YAGEO -> Murata; Part Number CC0402KPX5R8BB225 -> GRT155R61E225KE13D
- Y1: Load Capacitance 12pF -> 12p
Changed lines of the file:
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@@
 			)
 		)
-		(property "Manufactorer" "YAGEO"
+		(property "Manufactorer" "Murata"
 			(at 191.77 43.18 0)
 			(effects
@@
 			)
 		)
-		(property "Part Number" "CC0402KPX5R8BB225"
+		(property "Part Number" "GRT155R61E225KE13D"
 			(at 191.77 43.18 0)
 			(effects
@@
 			)
 		)
-		(property "Manufactorer" "YAGEO"
+		(property "Manufactorer" "Murata"
 			(at 179.07 43.18 0)
 			(effects
@@
 			)
 		)
-		(property "Part Number" "CC0402KPX5R8BB225"
+		(property "Part Number" "GRT155R61E225KE13D"
 			(at 179.07 43.18 0)
 			(effects
@@
 			)
 		)
-		(property "Manufactorer" "YAGEO"
+		(property "Manufactorer" "Murata"
 			(at 116.84 129.54 0)
 			(effects
@@
 			)
 		)
-		(property "Part Number" "CC0402KPX5R8BB225"
+		(property "Part Number" "GRT155R61E225KE13D"
 			(at 116.84 129.54 0)
 			(effects
@@
 			)
 		)
-		(property "Manufactorer" "YAGEO"
+		(property "Manufactorer" "Murata"
 			(at 128.27 129.54 0)
 			(effects
@@
 			)
 		)
-		(property "Part Number" "CC0402KPX5R8BB225"
+		(property "Part Number" "GRT155R61E225KE13D"
 			(at 128.27 129.54 0)
 			(effects
@@
 			)
 		)
-		(property "Load Capacitance" "12pF"
+		(property "Load Capacitance" "12p"
 			(at 53.34 161.29 0)
 			(effects
