File: power.kicad_sch (KiCad schematic)
At the start: 25 parts, among them U7 AP63205WU, U8 AP63203WU

Commit message: replace flash memory with SD flash memory; move SPI2 terminations closer to source
Parts:
- C32, C36: Part Number CC0402KRX7R7BB104 -> CC0402KRX5R8BB104; Voltage 16 -> 25
- C33, C37: Manufactorer Samsung -> Murata; Part Number CL21A106KBYQNNE -> GRM21BR61H106KE43K
- C34, C35, C38, C39: Part Number GRM21BC81C226ME44L -> GRM21BR61E226ME44K; Voltage 16 -> 25
- D2, D4: Part Number SK34SMA-3G -> BAT60JFILM; Voltage 40 -> 10
- D3, D5: Part Number SK34SMA-3G -> PMEG60T30ELRX; Voltage 40 -> 60
- L1, L2: footprint Project:IND_DFE322520FD-4R7M=P2_MUR -> Inductor_SMD:L_1210_3225Metric; Voltage (none) -> 2
- R20, R21: value 3k3 -> 1k5; Part Number RT0402BRD073K3L -> RT0402BRD071K5L
- R22: value 3k3 -> 1k2; Part Number RT0402BRD073K3L -> RT0402BRD071K2L
- R23: value 1k2 -> 680; Part Number RC0402FR-071K2L -> RC0402FR-07680RP
Changed lines of the file:
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@@
 		(fields_autoplaced yes)
 		(property "Reference" "R22"
-			(at 134.62 172.72 0)
+			(at 134.62 172.7199 0)
 			(effects
 				(font
@@
 			)
 		)
-		(property "Value" "3k3"
-			(at 134.62 175.26 0)
+		(property "Value" "1k2"
+			(at 134.62 175.2599 0)
 			(effects
 				(font
@@
 			)
 		)
-		(property "Part Number" "RT0402BRD073K3L"
+		(property "Part Number" "RT0402BRD071K2L"
 			(at 132.08 173.99 0)
 			(effects
@@
 			)
 		)
-		(property "Footprint" "Project:IND_DFE322520FD-4R7M=P2_MUR"
+		(property "Footprint" "Inductor_SMD:L_1210_3225Metric"
 			(at 114.3 55.88 0)
 			(effects
@@
 			)
 		)
-		(property "Datasheet" "~"
+		(property "Datasheet" "https://search.murata.co.jp/Ceramy/image/img/P02/J(E)TE243A-9104.pdf"
 			(at 114.3 55.88 0)
 			(effects
@@
 			)
 		)
+		(property "Voltage" "2"
+			(at 114.3 55.88 0)
+			(effects
+				(font
+					(size 1.27 1.27)
+				)
+				(hide yes)
+			)
+		)
 		(pin "2"
 		)
@@
 			)
 		)
-		(property "Voltage" "16"
+		(property "Voltage" "25"
 			(at 260.35 67.31 0)
 			(effects
@@
 			)
 		)
-		(property "Part Number" "GRM21BC81C226ME44L"
+		(property "Part Number" "GRM21BR61E226ME44K"
 			(at 260.35 67.31 0)
 			(effects
@@
 			)
 		)
-		(property "Datasheet" "https://www.infineon.com/dgdl/Infineon-BAT60ASERIES-DS-v01_01-en.pdf?fileId=db3a304313d846880113def70c9304a9"
+		(property "Datasheet" "https://assets.nexperia.com/documents/data-sheet/PMEG60T30ELR.pdf"
 			(at 185.42 124.46 0)
 			(effects
@@
 			)
 		)
-		(property "Part Number" "SK34SMA-3G"
+		(property "Part Number" "PMEG60T30ELRX"
 			(at 185.42 124.46 0)
 			(effects
@@
 			)
 		)
-		(property "Voltage" "40"
+		(property "Voltage" "60"
 			(at 185.42 124.46 0)
 			(effects
@@
 			)
 		)
-		(property "Datasheet" "https://www.infineon.com/dgdl/Infineon-BAT60ASERIES-DS-v01_01-en.pdf?fileId=db3a304313d846880113def70c9304a9"
+		(property "Datasheet" "https://www.st.com/content/ccc/resource/technical/document/datasheet/3d/d2/27/1d/20/e3/4d/48/CD00001944.pdf/files/CD00001944.pdf/jcr:content/translations/en.CD00001944.pdf"
 			(at 140.97 109.22 0)
 			(effects
@@
 			)
 		)
-		(property "Part Number" "SK34SMA-3G"
+		(property "Part Number" "BAT60JFILM"
 			(at 140.97 109.22 0)
 			(effects
@@
 			)
 		)
-		(property "Voltage" "40"
+		(property "Voltage" "10"
 			(at 140.97 109.22 0)
 			(effects
@@
 			)
 		)
-		(property "Voltage" "16"
+		(property "Voltage" "25"
 			(at 238.76 58.42 0)
 			(effects
@@
 			)
 		)
-		(property "Part Number" "CC0402KRX7R7BB104"
+		(property "Part Number" "CC0402KRX5R8BB104"
 			(at 238.76 58.42 0)
 			(effects
@@
 		(fields_autoplaced yes)
 		(property "Reference" "R23"
-			(at 153.67 172.72 0)
+			(at 153.67 172.7199 0)
 			(effects
 				(font
@@
 			)
 		)
-		(property "Value" "1k2"
-			(at 153.67 175.26 0)
+		(property "Value" "680"
+			(at 153.67 175.2599 0)
 			(effects
 				(font
@@
 			)
 		)
-		(property "Part Number" "RC0402FR-071K2L"
+		(property "Part Number" "RC0402FR-07680RP"
 			(at 151.13 173.99 0)
 			(effects
@@
 			)
 		)
-		(property "Manufactorer" "Samsung"
+		(property "Manufactorer" "Murata"
 			(at 69.85 64.77 0)
 			(effects
@@
 			)
 		)
-		(property "Part Number" "CL21A106KBYQNNE"
+		(property "Part Number" "GRM21BR61H106KE43K"
 			(at 69.85 64.77 0)
 			(effects
@@
 		(fields_autoplaced yes)
 		(property "Reference" "R21"
-			(at 101.6 172.72 0)
+			(at 101.6 172.7199 0)
 			(effects
 				(font
@@
 			)
 		)
-		(property "Value" "3k3"
-			(at 101.6 175.26 0)
+		(property "Value" "1k5"
+			(at 101.6 175.2599 0)
 			(effects
 				(font
@@
 			)
 		)
-		(property "Part Number" "RT0402BRD073K3L"
+		(property "Part Number" "RT0402BRD071K5L"
 			(at 99.06 173.99 0)
 			(effects
@@
 			)
 		)
-		(property "Manufactorer" "Samsung"
+		(property "Manufactorer" "Murata"
 			(at 204.47 63.5 0)
 			(effects
@@
 			)
 		)
-		(property "Part Number" "CL21A106KBYQNNE"
+		(property "Part Number" "GRM21BR61H106KE43K"
 			(at 204.47 63.5 0)
 			(effects
@@
 			)
 		)
-		(property "Voltage" "16"
+		(property "Voltage" "25"
 			(at 104.14 59.69 0)
 			(effects
@@
 			)
 		)
-		(property "Part Number" "CC0402KRX7R7BB104"
+		(property "Part Number" "CC0402KRX5R8BB104"
 			(at 104.14 59.69 0)
 			(effects
@@
 			)
 		)
-		(property "Footprint" "Project:IND_DFE322520FD-4R7M=P2_MUR"
+		(property "Footprint" "Inductor_SMD:L_1210_3225Metric"
 			(at 250.19 54.61 0)
 			(effects
@@
 			)
 		)
-		(property "Datasheet" "~"
+		(property "Datasheet" "https://search.murata.co.jp/Ceramy/image/img/P02/J(E)TE243A-0019.pdf"
 			(at 250.19 54.61 0)
 			(effects
@@
 			)
 		)
+		(property "Voltage" "2"
+			(at 250.19 54.61 0)
+			(effects
+				(font
+					(size 1.27 1.27)
+				)
+				(hide yes)
+			)
+		)
 		(pin "2"
 		)
@@
 			)
 		)
-		(property "Datasheet" "D26V0H1U2LP20-7"
+		(property "Datasheet" "https://www.diodes.com/assets/Datasheets/D26V0H1U2LP20.pdf"
 			(at 62.23 71.12 0)
 			(effects
@@
 			)
 		)
-		(property "Datasheet" "https://www.infineon.com/dgdl/Infineon-BAT60ASERIES-DS-v01_01-en.pdf?fileId=db3a304313d846880113def70c9304a9"
+		(property "Datasheet" "https://assets.nexperia.com/documents/data-sheet/PMEG60T30ELR.pdf"
 			(at 185.42 109.22 0)
 			(effects
@@
 			)
 		)
-		(property "Part Number" "SK34SMA-3G"
+		(property "Part Number" "PMEG60T30ELRX"
 			(at 185.42 109.22 0)
 			(effects
@@
 			)
 		)
-		(property "Voltage" "40"
+		(property "Voltage" "60"
 			(at 185.42 109.22 0)
 			(effects
@@
 			)
 		)
-		(property "Voltage" "16"
+		(property "Voltage" "25"
 			(at 130.81 68.58 0)
 			(effects
@@
 			)
 		)
-		(property "Part Number" "GRM21BC81C226ME44L"
+		(property "Part Number" "GRM21BR61E226ME44K"
 			(at 130.81 68.58 0)
 			(effects
@@
 			)
 		)
-		(property "Voltage" "16"
+		(property "Voltage" "25"
 			(at 125.73 68.58 0)
 			(effects
@@
 			)
 		)
-		(property "Part Number" "GRM21BC81C226ME44L"
+		(property "Part Number" "GRM21BR61E226ME44K"
 			(at 125.73 68.58 0)
 			(effects
@@
 			)
 		)
-		(property "Datasheet" "~"
+		(property "Datasheet" "https://optoelectronics.liteon.com/upload/download/DS22-2000-223/LTST-C191KRKT.PDF"
 			(at 76.2 166.37 0)
 			(effects
@@
 			)
 		)
-		(property "Datasheet" "~"
+		(property "Datasheet" "https://mm.digikey.com/Volume0/opasdata/d220001/medias/docus/1294/LTST-C191GKT.pdf"
 			(at 132.08 166.37 0)
 			(effects
@@
 			)
 		)
-		(property "Datasheet" "~"
+		(property "Datasheet" "https://mm.digikey.com/Volume0/opasdata/d220001/medias/docus/1294/LTST-C191GKT.pdf"
 			(at 151.13 166.37 0)
 			(effects
@@
 		(fields_autoplaced yes)
 		(property "Reference" "R20"
-			(at 78.74 172.72 0)
+			(at 78.74 172.7199 0)
 			(effects
 				(font
@@
 			)
 		)
-		(property "Value" "3k3"
-			(at 78.74 175.26 0)
+		(property "Value" "1k5"
+			(at 78.74 175.2599 0)
 			(effects
 				(font
@@
 			)
 		)
-		(property "Part Number" "RT0402BRD073K3L"
+		(property "Part Number" "RT0402BRD071K5L"
 			(at 76.2 173.99 0)
 			(effects
@@
 			)
 		)
-		(property "Datasheet" "~"
+		(property "Datasheet" "https://optoelectronics.liteon.com/upload/download/DS22-2000-223/LTST-C191KRKT.PDF"
 			(at 99.06 166.37 0)
 			(effects
@@
 			)
 		)
-		(property "Voltage" "16"
+		(property "Voltage" "25"
 			(at 265.43 67.31 0)
 			(effects
@@
 			)
 		)
-		(property "Part Number" "GRM21BC81C226ME44L"
+		(property "Part Number" "GRM21BR61E226ME44K"
 			(at 265.43 67.31 0)
 			(effects
@@
 			)
 		)
-		(property "Datasheet" "https://www.infineon.com/dgdl/Infineon-BAT60ASERIES-DS-v01_01-en.pdf?fileId=db3a304313d846880113def70c9304a9"
+		(property "Datasheet" "https://www.st.com/content/ccc/resource/technical/document/datasheet/3d/d2/27/1d/20/e3/4d/48/CD00001944.pdf/files/CD00001944.pdf/jcr:content/translations/en.CD00001944.pdf"
 			(at 140.97 124.46 0)
 			(effects
@@
 			)
 		)
-		(property "Part Number" "SK34SMA-3G"
+		(property "Part Number" "BAT60JFILM"
 			(at 140.97 124.46 0)
 			(effects
@@
 			)
 		)
-		(property "Voltage" "40"
+		(property "Voltage" "10"
 			(at 140.97 124.46 0)
 			(effects

Commit message: relabel components by sheet and block
Parts:
- L1, L2: Amps (none) -> 2; Voltage 2 -> (none)
- U7: Amps (none) -> 2; Voltage (none) -> 5
- U8: Amps (none) -> 2; Voltage (none) -> 3
- renumbered C32 to C34, C33 to C35, C34 to C36, C35 to C37, C36 to C38, C37 to C39, C38 to C40, C39 to C41, D4 to D3, D3 to D4, R20 to R23, R21 to R24, R22 to R25, R23 to R26

Commit message: remove blind vias and use 0201 resistors
Parts:
- C34, C38: footprint Capacitor_SMD:C_0402_1005Metric -> Project:C_0201_0603Metric; Manufactorer YAGEO -> Murata; Part Number CC0402KRX5R8BB104 -> GRM033R61E104KE14J
- R23, R24: footprint Resistor_SMD:R_0402_1005Metric -> Project:R_0201_0603Metric; Part Number RT0402BRD071K5L -> RC0201FR-071K5L
- R25: footprint Resistor_SMD:R_0402_1005Metric -> Project:R_0201_0603Metric; Part Number RT0402BRD071K2L -> RC0201FR-071K2L
- R26: footprint Resistor_SMD:R_0402_1005Metric -> Project:R_0201_0603Metric; Part Number RC0402FR-07680RP -> RC0201FR-07680RL
Changed lines of the file:
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@@
 			)
 		)
-		(property "Footprint" "Resistor_SMD:R_0402_1005Metric"
+		(property "Footprint" "Project:R_0201_0603Metric"
 			(at 130.302 173.99 90)
 			(effects
@@
 			)
 		)
-		(property "Part Number" "RT0402BRD071K2L"
+		(property "Part Number" "RC0201FR-071K2L"
 			(at 132.08 173.99 0)
 			(effects
@@
 			)
 		)
-		(property "Footprint" "Capacitor_SMD:C_0402_1005Metric"
+		(property "Footprint" "Project:C_0201_0603Metric"
 			(at 239.7252 62.23 0)
 			(effects
@@
 			)
 		)
-		(property "Manufactorer" "YAGEO"
+		(property "Manufactorer" "Murata"
 			(at 238.76 58.42 0)
 			(effects
@@
 			)
 		)
-		(property "Part Number" "CC0402KRX5R8BB104"
+		(property "Part Number" "GRM033R61E104KE14J"
 			(at 238.76 58.42 0)
 			(effects
@@
 			)
 		)
-		(property "Footprint" "Resistor_SMD:R_0402_1005Metric"
+		(property "Footprint" "Project:R_0201_0603Metric"
 			(at 149.352 173.99 90)
 			(effects
@@
 			)
 		)
-		(property "Part Number" "RC0402FR-07680RP"
+		(property "Part Number" "RC0201FR-07680RL"
 			(at 151.13 173.99 0)
 			(effects
@@
 			)
 		)
-		(property "Footprint" "Resistor_SMD:R_0402_1005Metric"
+		(property "Footprint" "Project:R_0201_0603Metric"
 			(at 97.282 173.99 90)
 			(effects
@@
 			)
 		)
-		(property "Part Number" "RT0402BRD071K5L"
+		(property "Part Number" "RC0201FR-071K5L"
 			(at 99.06 173.99 0)
 			(effects
@@
 			)
 		)
-		(property "Footprint" "Capacitor_SMD:C_0402_1005Metric"
+		(property "Footprint" "Project:C_0201_0603Metric"
 			(at 105.1052 63.5 0)
 			(effects
@@
 			)
 		)
-		(property "Manufactorer" "YAGEO"
+		(property "Manufactorer" "Murata"
 			(at 104.14 59.69 0)
 			(effects
@@
 			)
 		)
-		(property "Part Number" "CC0402KRX5R8BB104"
+		(property "Part Number" "GRM033R61E104KE14J"
 			(at 104.14 59.69 0)
 			(effects
@@
 			)
 		)
-		(property "Footprint" "Resistor_SMD:R_0402_1005Metric"
+		(property "Footprint" "Project:R_0201_0603Metric"
 			(at 74.422 173.99 90)
 			(effects
@@
 			)
 		)
-		(property "Part Number" "RT0402BRD071K5L"
+		(property "Part Number" "RC0201FR-071K5L"
 			(at 76.2 173.99 0)
 			(effects

Commit message: double check BOM
Parts:
- D1: Voltage 40 -> 26
- D4, D5: value PMEG60T30ELRX -> PMEG3030CERX; Part Number PMEG60T30ELRX -> PMEG3030CERX; Voltage 60 -> 30
- D6, D7: Voltage (none) -> 2
- D8, D9: Voltage (none) -> 2.1
- L1, L2: Tolerance (none) -> 20%
Changed lines of the file:
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@@
 			)
 		)
+		(property "Tolerance" "20%"
+			(at 114.3 55.88 0)
+			(effects
+				(font
+					(size 1.27 1.27)
+				)
+				(hide yes)
+			)
+		)
 		(pin "2"
 		)
@@
 			)
 		)
-		(property "Value" "PMEG60T30ELRX"
+		(property "Value" "PMEG3030CERX"
 			(at 185.42 121.92 0)
 			(effects
@@
 			)
 		)
-		(property "Part Number" "PMEG60T30ELRX"
+		(property "Part Number" "PMEG3030CERX"
 			(at 185.42 124.46 0)
 			(effects
@@
 			)
 		)
-		(property "Voltage" "60"
+		(property "Voltage" "30"
 			(at 185.42 124.46 0)
 			(effects
@@
 			)
 		)
+		(property "Tolerance" "20%"
+			(at 250.19 54.61 0)
+			(effects
+				(font
+					(size 1.27 1.27)
+				)
+				(hide yes)
+			)
+		)
 		(pin "2"
 		)
@@
 			)
 		)
-		(property "Voltage" "40"
+		(property "Voltage" "26"
 			(at 62.23 71.12 0)
 			(effects
@@
 			)
 		)
-		(property "Value" "PMEG60T30ELRX"
+		(property "Value" "PMEG3030CERX"
 			(at 185.42 106.68 0)
 			(effects
@@
 			)
 		)
-		(property "Part Number" "PMEG60T30ELRX"
+		(property "Part Number" "PMEG3030CERX"
 			(at 185.42 109.22 0)
 			(effects
@@
 			)
 		)
-		(property "Voltage" "60"
+		(property "Voltage" "30"
 			(at 185.42 109.22 0)
 			(effects
@@
 			)
 		)
+		(property "Voltage" "2"
+			(at 76.2 166.37 0)
+			(effects
+				(font
+					(size 1.27 1.27)
+				)
+				(hide yes)
+			)
+		)
 		(pin "1"
 		)
@@
 			)
 		)
+		(property "Voltage" "2.1"
+			(at 132.08 166.37 0)
+			(effects
+				(font
+					(size 1.27 1.27)
+				)
+				(hide yes)
+			)
+		)
 		(pin "1"
 		)
@@
 			)
 		)
+		(property "Voltage" "2.1"
+			(at 151.13 166.37 0)
+			(effects
+				(font
+					(size 1.27 1.27)
+				)
+				(hide yes)
+			)
+		)
 		(pin "1"
 		)
@@
 			(at 99.06 166.37 0)
 			(effects
+				(font
+					(size 1.27 1.27)
+				)
+				(hide yes)
+			)
+		)
+		(property "Voltage" "2"
+			(at 99.06 166.37 0)
+			(effects
