File: peripherals.kicad_sch (KiCad schematic)
At the start: 35 parts, among them U2 AT7456E, U3 TXU0304PWR, U4 ICM-42688-P, U5 MT29F2G01ABAGDWB-IT_G, U6 DPS310XTSA1, Y2 27MHz

Commit message: replace flash memory with SD flash memory; move SPI2 terminations closer to source
Parts:
- removed R18: 5k1, Resistor_SMD:R_0402_1005Metric, symbol Device:R
- removed U5: MT29F2G01ABAGDWB-IT_G, Project:SON127P600X800X65-8N, symbol Project_Library:MT29F2G01ABAGDWB-IT_G
- added R34: 100k, Resistor_SMD:R_0402_1005Metric, symbol Device:R
- added R35, R40, R41: 22, Resistor_SMD:R_0402_1005Metric, symbol Device:R
- added U5: XTSD04G, Package_LGA:LGA-8_8x6mm_P1.27mm, symbol Memory_Flash:XTSD04G
- C15, C16: Part Number GRM21BC81C226ME44L -> GRM21BR61E226ME44K; Voltage 16 -> 25
- C17, C25, C28, C30, C52, C53: Part Number GRM188C71C225KE11D -> GRM188R61E225KA12D; Voltage 16 -> 25
- C18, C19, C20, C21, C22, C23, C24, C26, C27, C29, C31: Part Number CC0402KRX7R7BB104 -> CC0402KRX5R8BB104; Voltage 16 -> 25
Connections:
- net +3V3: now also U5.8 (VDD); no longer U6.2 (~{CSB})
- net GND: now also R34.2, U5.4 (VSS); no longer U6.5 (SDO)
- net SPI2_CS_FLASH: now also U5.2 (SD3/~{CS})
- net SPI2_MISO_4V: now also R41.1; no longer U2.11 (SDOUT)
- net SPI2_MOSI: now also U5.5 (CMD/DI)
- net SPI2_MOSI_4V: now also R35.2; no longer U3.12 (B2Y)
- net SPI2_SCK: now also U5.3 (CLK)
- net SPI2_SCK_4V: now also R40.2; no longer U3.11 (B3Y)
- net at R19.1: now also U5.6 (SD0/DO)
- new net: R40.1, U3.11 (B3Y)
- new net: R35.1, U3.12 (B2Y)
- new net: R41.2, U2.11 (SDOUT)
- new net: R34.1, U6.5 (SDO)
- no-connect marks 15 -> 17
Other:
- moved on the sheet: C22, C23, C27, C28, C52, C53, R15, R16, R19, U3

Commit message: relabel components by sheet and block
Parts:
- removed Y2: 27MHz, Crystal:Crystal_SMD_0603-2Pin_6.0x3.5mm, symbol Device:Crystal
- added Y2: 27MHz, Project:XTAL_ECS-270-20-30B-TR, symbol Device:Crystal_GND24
- U3: renamed from U5; Note CSNP4GCR01-AMW (Creat Storage World); MKDV4GCL-AB (MK); ZDS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 -> alternates: CSNP4GCR01-AMW (Creat Storage World) or MKDV4GC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
- renumbered C27 to C22, C28 to C23, C53 to C24, C22 to C25, C23 to C26, C52 to C27, C24 to C28, C25 to C29, C26 to C30, C29 to C31, C30 to C32, C31 to C33, R41 to R12, R12 to R13, R13 to R14, R14 to R15, R19 to R16, R35 to R17, R40 to R18, R15 to R19, R16 to R20, R17 to R21, R34 to R22, U3 to U4, U4 to U5
Connections:
- net GND: now also Y2.2, Y2.4
- net XFB: now reaches U2.6 (XFB)
- net XFB: now also Y2.1
- net CLKIN: now reaches U2.5 (CLKIN)
- net CLKIN: now also Y2.3
Other:
- moved on the sheet: C17, C18

Commit message: remove blind vias and use 0201 resistors
Parts:
- C17, C23, C24, C27, C29, C32: footprint Capacitor_SMD:C_0603_1608Metric -> Capacitor_SMD:C_0402_1005Metric; Manufactorer Murata -> YAGEO; Part Number GRM188R61E225KA12D -> CC0402KPX5R8BB225
- C18, C19, C20, C21, C22, C25, C26, C28, C30, C31, C33: footprint Capacitor_SMD:C_0402_1005Metric -> Project:C_0201_0603Metric; Manufactorer YAGEO -> Murata; Part Number CC0402KRX5R8BB104 -> GRM033R61E104KE14J
- R10, R11: footprint Resistor_SMD:R_0402_1005Metric -> Project:R_0201_0603Metric; Part Number RC0402FR-0775RP -> RC0201FR-0775RL
- R12, R16, R17, R18, R19, R21: footprint Resistor_SMD:R_0402_1005Metric -> Project:R_0201_0603Metric; Part Number RC0402FR-0722RP -> RC0201FR-0722RL
- R13, R14, R15: footprint Resistor_SMD:R_0402_1005Metric -> Project:R_0201_0603Metric
- R20: footprint Resistor_SMD:R_0402_1005Metric -> Project:R_0201_0603Metric; Part Number RC0402FR-075K1L -> RC0201FR-075K1L
- R22: footprint Resistor_SMD:R_0402_1005Metric -> Project:R_0201_0603Metric; Part Number RC0402FR-07100KL -> RC0201FR-07100KL; Tolerance (none) -> 1%

Commit message: double check BOM
Parts:
- C17, C23, C24, C27, C29, C32: Manufactorer YAGEO -> Murata; Part Number CC0402KPX5R8BB225 -> GRT155R61E225KE13D
- R13, R14, R15: Part Number RC0402FR-071KL -> RC0201FR-071KL
- U3: value XTSD04G -> CSNP4GCR01-AMW; Manufactorer XTX -> Create Storage World; Note alternates: CSNP4GCR01-AMW (Creat Storage World) or MKDV4GCL-AB (MK) or ZDSD04G (Zetta) -> alternates: CSNP4GCR01-AMW (Creat Storage World) or MKDV4GCL-AB (MK) or ZDSD04G (Zetta) or XTSD04G (XTX); Part Number XTSD04G -> CSNP4GCR01-AMW
- Y2: Load Capacitance (none) -> 18p
Changed lines of the file:
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@@
 			)
 		)
-		(property "Manufactorer" "YAGEO"
+		(property "Manufactorer" "Murata"
 			(at 255.27 38.1 0)
 			(effects
@@
 			)
 		)
-		(property "Part Number" "CC0402KPX5R8BB225"
+		(property "Part Number" "GRT155R61E225KE13D"
 			(at 255.27 38.1 0)
 			(effects
@@
 			)
 		)
-		(property "Manufactorer" "YAGEO"
+		(property "Manufactorer" "Murata"
 			(at 22.86 115.57 0)
 			(effects
@@
 			)
 		)
-		(property "Part Number" "CC0402KPX5R8BB225"
+		(property "Part Number" "GRT155R61E225KE13D"
 			(at 22.86 115.57 0)
 			(effects
@@
 			)
 		)
-		(property "Part Number" "RC0402FR-071KL"
+		(property "Part Number" "RC0201FR-071KL"
 			(at 123.19 81.28 0)
 			(effects
@@
 			)
 		)
-		(property "Value" "XTSD04G"
+		(property "Value" "CSNP4GCR01-AMW"
 			(at 245.11 49.5299 0)
 			(effects
@@
 			)
 		)
-		(property "Datasheet" "https://datasheet.lcsc.com/lcsc/2005251034_XTX-XTSD08GLGEAG_C558840.pdf"
+		(property "Datasheet" "https://www.lcsc.com/datasheet/lcsc_datasheet_2102221705_Creat-Storage-World-CSNP4GCR01-AMW_C2691596.pdf"
 			(at 238.76 48.26 0)
 			(effects
@@
 			)
 		)
-		(property "Manufactorer" "XTX"
+		(property "Manufactorer" "Create Storage World"
 			(at 236.22 48.26 0)
 			(effects
@@
 			)
 		)
-		(property "Note" "alternates: CSNP4GCR01-AMW (Creat Storage World) or  MKDV4GCL-AB (MK) or ZDSD04G (Zetta) "
+		(property "Note" "alternates: CSNP4GCR01-AMW (Creat Storage World) or  MKDV4GCL-AB (MK) or ZDSD04G (Zetta)  or XTSD04G (XTX)"
 			(at 236.22 67.818 0)
 			(effects
@@
 			)
 		)
-		(property "Part Number" "XTSD04G"
+		(property "Part Number" "CSNP4GCR01-AMW"
 			(at 236.22 48.26 0)
 			(effects
@@
 			)
 		)
-		(property "Part Number" "RC0402FR-071KL"
+		(property "Part Number" "RC0201FR-071KL"
 			(at 114.3 81.28 0)
 			(effects
@@
 			)
 		)
-		(property "Manufactorer" "YAGEO"
+		(property "Manufactorer" "Murata"
 			(at 144.78 119.38 0)
 			(effects
@@
 			)
 		)
-		(property "Part Number" "CC0402KPX5R8BB225"
+		(property "Part Number" "GRT155R61E225KE13D"
 			(at 144.78 119.38 0)
 			(effects
@@
 			)
 		)
-		(property "Manufactorer" "YAGEO"
+		(property "Manufactorer" "Murata"
 			(at 144.78 160.02 0)
 			(effects
@@
 			)
 		)
-		(property "Part Number" "CC0402KPX5R8BB225"
+		(property "Part Number" "GRT155R61E225KE13D"
 			(at 144.78 160.02 0)
 			(effects
@@
 			)
 		)
-		(property "Manufactorer" "YAGEO"
+		(property "Manufactorer" "Murata"
 			(at 269.24 125.73 0)
 			(effects
@@
 			)
 		)
-		(property "Part Number" "CC0402KPX5R8BB225"
+		(property "Part Number" "GRT155R61E225KE13D"
 			(at 269.24 125.73 0)
 			(effects
@@
 			)
 		)
-		(property "Manufactorer" "YAGEO"
+		(property "Manufactorer" "Murata"
 			(at 30.48 36.83 0)
 			(effects
@@
 			)
 		)
-		(property "Part Number" "CC0402KPX5R8BB225"
+		(property "Part Number" "GRT155R61E225KE13D"
 			(at 30.48 36.83 0)
 			(effects
@@
 			)
 		)
+		(property "Load Capacitance" "18p"
+			(at 33.02 71.12 0)
+			(effects
+				(font
+					(size 1.27 1.27)
+				)
+				(hide yes)
+			)
+		)
 		(pin "1"
 		)
@@
 			)
 		)
-		(property "Part Number" "RC0402FR-071KL"
+		(property "Part Number" "RC0201FR-071KL"
 			(at 132.08 81.28 0)
 			(effects

Commit message: remove soldermask bridges for IMU to faciliate assembly by PCBWAY
Parts:
- U5: footprint Project:PQFN50P300X250X97-14N -> Project:LGA-14_3x2.5mm_P0.5mm_LayoutBorder3x4y_no_mask_bridges
Changed lines of the file:
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@@
 			)
 		)
-		(property "Footprint" "Project:PQFN50P300X250X97-14N"
+		(property "Footprint" "Project:LGA-14_3x2.5mm_P0.5mm_LayoutBorder3x4y_no_mask_bridges"
 			(at 77.47 167.64 0)
 			(effects
